Commit message: Add boxes under and in front of the arm

File: src/irb1200_ros2_gazebo/urdf/irb1200.urdf.xacro (robot description, xacro)
@@ -67,7 +67,66 @@
   <!-- CELL LAYOUT N1) ABB IRB1200 Robot alone: -->
   <xacro:if value="${cell_layout_1}">
-    <joint name="world-base_link-fixed" type="fixed">
+    <!-- <joint name="world-base_link-fixed" type="fixed">
       <parent link="world"/>
       <child link="base_link"/>
+    </joint> -->
+    <link name='irb120_block'>
+      <inertial>
+        <origin xyz="0 0 0" rpy="0 0 0"/>
+        <mass value="100"/>
+        <inertia ixx="0.01"  ixy="0"  ixz="0" iyy="0.01" iyz="0" izz="0.01" />
+      </inertial>
+      <collision name='collision'>
+        <origin xyz="0 0 0" rpy=" 0 0 0"/>
+        <geometry>
+          <box size = "0.2 0.2 0.5"/>
+        </geometry>
+      </collision>
+      <visual name='chassis_visual'>
+        <origin xyz="0 0 0" rpy=" 0 0 0"/>
+        <geometry>
+          <box size = "0.2 0.2 0.5"/>
+        </geometry>
+        <material name="red">
+          <color rgba="1 0 0 1"/>
+        </material>
+      </visual>
+    </link>
+    <joint name="world_joint" type="fixed">
+      <parent link="world" />
+      <child link = "irb120_block" />
+      <origin xyz="0.0 0.0 0.25" rpy="0.0 0.0 0.0" />
+    </joint>
+    <joint name="block-base" type="fixed">
+      <parent link="irb120_block" />
+      <child link = "base_link" />
+      <origin xyz="0.0 0.0 0.255" rpy="0.0 0.0 0.0" />
+    </joint>
+    <link name='table'>
+      <inertial>
+        <origin xyz="0 0 0" rpy="0 0 0"/>
+        <mass value="100"/>
+        <inertia ixx="0.01"  ixy="0"  ixz="0" iyy="0.01" iyz="0" izz="0.01" />
+      </inertial>
+      <collision name='collision'>
+        <origin xyz="0 0 0" rpy=" 0 0 0"/>
+        <geometry>
+          <box size = "0.5 1.0 0.7"/>
+        </geometry>
+      </collision>
+      <visual name='chassis_visual'>
+        <origin xyz="0 0 0" rpy=" 0 0 0"/>
+        <geometry>
+          <box size = "0.5 1.0 0.7"/>
+        </geometry>
+        <material name="black">
+          <color rgba="1 0 0 1"/>
+        </material>
+      </visual>
+    </link>
+    <joint name="table_world" type="fixed">
+      <parent link="world" />
+      <child link = "table" />
+      <origin xyz="0.7 0.0 0.35" rpy="0.0 0.0 0.0" />
     </joint>
   </xacro:if>

File: src/simulation/urdf/pippo.urdf (robot description, URDF)
Before this commit: robot pippo, 5 links, 4 joints
Links:
- added link box_link, mass 1; collision box size=0.15 0.15 0.15; visual box size=0.15 0.15 0.15
- added link platform_link, mass 1; collision box size=0.40 0.40 0.01; visual box size=0.40 0.40 0.01
Joints:
- added joint box_joint: type floating, parent platform_link, child box_link, origin xyz=0 0 0.5 rpy=0. 0. 0., axis 0 0 1, limit lower=-0.05 upper=0.24 effort=10000.0 velocity=0.5
- added joint platform_joint: type fixed, parent pippo/lidar_link, child platform_link, origin xyz=0 0 0.05 rpy=0. 0. 0., axis 0 0 1, limit lower=-0.05 upper=0.24 effort=10000.0 velocity=0.5
