Commit message: - Add irb120 robot - Put correct robot launch file in pippo.launch.py  - Fix ros2_execution.py programs search path

File: src/simulation/urdf/pippo.urdf (robot description, URDF)
Before this commit: robot pippo, 7 links, 6 joints
Links:
- removed link box_link
Joints:
- removed joint box_joint

Commit message: - Add non-worning plugin to add a joint between the box and the robot's platform

File: src/simulation/urdf/pippo.urdf (robot description, URDF)
Before this commit: robot pippo, 6 links, 5 joints
Links:
- removed link platform_link
- added link pippo/platform_link, mass 1; collision box size=0.40 0.40 0.01; visual box size=0.40 0.40 0.01
Joints:
- joint platform_joint: child platform_link -> pippo/platform_link

Commit message: Fix everything

File: src/simulation/urdf/pippo.urdf (robot description, URDF)
Before this commit: robot pippo, 6 links, 5 joints
Links:
- link pippo/platform_link: mass 1 -> 0.125
Joints:
- joint lidar_joint: axis (none) -> 0 1 0
