Commit message: - Change robot name - Run without Gazebo GUI

File: src/simulation/urdf/robot.urdf (robot description, URDF)
Before this commit: robot pippo, 7 links, 6 joints
Links:
- removed link pippo/base_footprint
- removed link pippo/base_link
- removed link pippo/gnss_link
- removed link pippo/imu_link
- removed link pippo/lidar_link
- removed link pippo/platform_link
- added link robot/base_footprint
- added link robot/base_link; collision box size=${base_length} ${base_width} ${base_height}; visual box size=${base_length} ${base_width} ${base_height}
- added link robot/gnss_link, mass 0.005; collision sphere radius=0.05; visual sphere radius=0.05
- added link robot/imu_link; collision box size=0.1 0.1 0.1; visual box size=0.1 0.1 0.1
- added link robot/lidar_link, mass 0.125; collision cylinder length=0.055 radius=0.0508; visual cylinder length=0.055 radius=0.0508
- added link robot/platform_link, mass 0.125; collision box size=0.40 0.40 0.01; visual box size=0.40 0.40 0.01
Joints:
- joint base_joint: child pippo/base_footprint -> robot/base_footprint; parent pippo/base_link -> robot/base_link
- joint caster_joint: parent pippo/base_link -> robot/base_link
- joint gnss_joint: child pippo/gnss_link -> robot/gnss_link; parent pippo/base_link -> robot/base_link
- joint imu_joint: child pippo/imu_link -> robot/imu_link; parent pippo/base_link -> robot/base_link
- joint lidar_joint: child pippo/lidar_link -> robot/lidar_link; parent pippo/base_link -> robot/base_link
- joint platform_joint: child pippo/platform_link -> robot/platform_link; parent pippo/lidar_link -> robot/lidar_link
