Commit message: Add example script

File: src/irb120_ros2_gazebo/urdf/irb120.urdf.xacro (robot description, xacro)
@@ -120,5 +120,5 @@
         <origin xyz="0 0 0" rpy=" 0 0 0"/>
         <geometry>
-          <box size = "0.2 0.2 0.5"/>
+          <box size = "0.2 0.2 0.3"/>
         </geometry>
       </collision>
@@ -126,5 +126,5 @@
         <origin xyz="0 0 0" rpy=" 0 0 0"/>
         <geometry>
-          <box size = "0.2 0.2 0.5"/>
+          <box size = "0.2 0.2 0.3"/>
         </geometry>
         <material name="red">
@@ -136,10 +136,10 @@
       <parent link="world" />
       <child link = "irb120_block" />
-      <origin xyz="0.0 0.0 0.25" rpy="0.0 0.0 0.0" />
+      <origin xyz="0.0 0.0 0.15" rpy="0.0 0.0 0.0" />
     </joint>
     <joint name="block-base" type="fixed">
       <parent link="irb120_block" />
       <child link = "base_link" />
-      <origin xyz="0.0 0.0 0.255" rpy="0.0 0.0 0.0" />
+      <origin xyz="0.0 0.0 0.151" rpy="0.0 0.0 0.0" />
     </joint>
     <link name='table'>
@@ -152,5 +152,5 @@
         <origin xyz="0 0 0" rpy=" 0 0 0"/>
         <geometry>
-          <box size = "0.5 1.0 0.7"/>
+          <box size = "0.5 1.0 0.5"/>
         </geometry>
       </collision>
@@ -158,5 +158,5 @@
         <origin xyz="0 0 0" rpy=" 0 0 0"/>
         <geometry>
-          <box size = "0.5 1.0 0.7"/>
+          <box size = "0.5 1.0 0.5"/>
         </geometry>
         <material name="black">
@@ -168,5 +168,5 @@
       <parent link="world" />
       <child link = "table" />
-      <origin xyz="0.7 0.0 0.35" rpy="0.0 0.0 0.0" />
+      <origin xyz="0.7 0.0 0.25" rpy="0.0 0.0 0.0" />
     </joint>
   </xacro:if>

File: src/ros2_grasping/urdf/box.urdf (robot description, URDF)
Before this commit: robot box, 1 links, 0 joints
Links:
- link box: mass 0.1 -> 0.001

File: src/simulation/urdf/pippo.urdf (robot description, URDF)
Before this commit: robot pippo, 6 links, 5 joints
Links:
- added link caster_link, mass 0.5; collision sphere radius=0.055; visual sphere radius=0.055
Joints:
- added joint caster_joint: type continuous, parent pippo/base_link, child caster_link, origin xyz=0.12 0 -0.105 rpy=0 0 0, axis 1 1 0
- joint platform_joint: axis 0 0 1 -> (none); limit lower=-0.05 upper=0.24 effort=10000.0 velocity=0.5 -> (none); origin xyz=0 0 0.05 rpy=0. 0. 0. -> xyz=0 0 0.015 rpy=0. 0. 0.
